Commit message: Correct the arms base model and refactor

File: arctos_description/urdf/arctos.xacro (robot description, xacro)
@@ -1,117 +1,20 @@
 <?xml version="1.0"?>
 <robot name="arctos" xmlns:xacro="http://www.ros.org/wiki/xacro">
-  <xacro:include filename="$(find arctos_description)/urdf/common/materials.xacro" />
-  <xacro:include filename="$(find arctos_description)/urdf/common/joint_link.xacro" />
-  <xacro:include filename="$(find arctos_description)/urdf/arctos_ros2_control.xacro" />
-  <xacro:include filename="$(find arctos_description)/urdf/arctos_gripper.xacro" />
+  <xacro:arg name="prefix" default="" />
+  <xacro:arg name="include_gripper" default="false" />
+  <xacro:arg name="use_hardware" default="false" />
+  <xacro:include filename="$(find arctos_description)/urdf/arctos_arm.xacro" />
   <link name="world" />
-  <joint name="world_joint" type="fixed">
-      <parent link="world"/>
-      <child link="base_link"/>
+  <joint name="$(arg prefix)world_joint" type="fixed">
+    <parent link="world" />
+    <child link="$(arg prefix)base_link" />
+    <origin xyz="0 0 0" rpy="0 0 0" />
   </joint>
-  <!-- Define all links -->
-  <xacro:arctos_link
-    name="base_link"
-    origin_xyz="0 0 0" origin_rpy="0 0 0"
-    material_name="white"
-    inertia_origin_xyz="0.0009375030874740357 0.047087016508753216 0.06663230338123677"
-    inertia_origin_rpy="0 0 0"
-    mass="2.3"
-    ixx="0.0143" iyy="0.0055" izz="0.015" ixy="0.0" iyz="0.0" ixz="0.0"
-  />
-  <xacro:arctos_link
-    name="Link_1_1"
-    origin_xyz="-0.0 -0.000 -0.1126" origin_rpy="0 0 0"
-    material_name="white"
-    inertia_origin_xyz="-0.0088 -0.0005 ${0.2116-0.1126}" inertia_origin_rpy="0 0 0"
-    mass="3.0396"
-    ixx="0.0143" iyy="${0.0168*0.96536}" izz="${0.0084*0.96082}" ixy="${0.0143*-0.03956}"
-    ixz="${0.0143*-0.11546}" iyz="${0.0168*0.25198}"
-  />
-  <xacro:arctos_link
-    name="Link_2_1"
-    origin_xyz="0.0 0.020356 -0.2876" origin_rpy="0 0 0"
-    material_name="white"
-    inertia_origin_xyz="0.0042 ${-0.0098+0.020356} ${0.4174-0.2876}" inertia_origin_rpy="0 0 0"
-    mass="2.527"
-    ixx="${0.0282*0.99851}" iyy="${0.03*0.99865}" izz="${0.0063*0.99982}" ixy="${0.0282*0.05146}"
-    iyz="${0.03*-0.00591}" ixz="${0.0282*-0.01813}"
-  />
-  <xacro:arctos_link
-    name="Link_3_1"
-    origin_xyz="-0.0 0.019045 -0.54864" origin_rpy="0 0 0"
-    material_name="white"
-    inertia_origin_xyz="0.00158 -0.053 0.009" inertia_origin_rpy="0 0 0"
-    mass="0.87"
-    ixx="${0.0028*0.99944}" iyy="${0.0011*0.98426}" izz="${0.0027*0.98428}" ixy="${0.0028*-0.02203}"
-    iyz="${0.001*-0.17481}" ixz="${0.0028*0.02507}"
-  />
-  <xacro:arctos_link
-    name="Link_4_1"
-    origin_xyz="0.0 0.1578 -0.5704" origin_rpy="0 0 0"
-    material_name="white"
-    inertia_origin_xyz="0.0 -0.0535 -0.001733" inertia_origin_rpy="0 0 0"
-    mass="1.006"
-    ixx="${0.0021*0.99726}" iyy="${0.0024*0.99801}" izz="${0.0032*0.99925}" ixy="${0.0021*-0.6305}"
-    iyz="${0.0024*0.00082}" ixz="${0.0021*0.03862}"
-  />
-  <xacro:arctos_link
-    name="Link_5_1"
-    origin_xyz="0.0 0.2832 -0.56856" origin_rpy="0 0 0"
-    material_name="white"
-    inertia_origin_xyz="-0.0007 -0.0142 -0.0008" inertia_origin_rpy="0 0 0"
-    mass="0.3344"
-    ixx="0.0002" iyy="0.0005" izz="0.0005" ixy="0.0" iyz="0.0" ixz="0.0"
-  />
-  <xacro:arctos_link
-    name="Link_6_1"
-    origin_xyz="0.0 0.323 -0.5685" origin_rpy="0 0 0"
-    material_name="white"
-    inertia_origin_xyz="-0.0 -0.0 0.0" inertia_origin_rpy="0.0 0.0 0.0"
-    mass="1e-3"
-    ixx="1e-3" iyy="1e-3" izz="1e-3" ixy="-0.0" iyz="0.0" ixz="0.0"
-  />
-  <xacro:arctos_joint
-    name="X_joint" type="revolute"
-    parent="base_link" child="Link_1_1"
-    origin_xyz="0.0 0.0 0.1126" origin_rpy="0 0 0"
-    axis_xyz="0.0 0.0 1.0"
-    limit_u="${pi}" limit_l="${-pi}" limit_e="24.3" limit_v="15.0"
-  />
-  <xacro:arctos_joint
-    name="Y_joint" type="revolute"
-    parent="Link_1_1" child="Link_2_1"
-    origin_xyz="0.0 -0.020356 ${0.2876-0.1126}" origin_rpy="0 0 0"
-    axis_xyz="1.0 -0.0 -0.0"
-    limit_u="2.18" limit_l="-0.96" limit_e="270.0" limit_v="1.4"
-  />
-  <xacro:arctos_joint
-    name="Z_joint" type="revolute"
-    parent="Link_2_1" child="Link_3_1"
-    origin_xyz="0.0 0.001365 0.261035" origin_rpy="0 0 0"
-    axis_xyz="1.0 -0.0 0.0"
-    limit_u="${70/180*pi}" limit_l="${-pi/2}" limit_e="97.0" limit_v="1.4"
-  />
-  <xacro:arctos_joint
-    name="A_joint" type="revolute"
-    parent="Link_3_1" child="Link_4_1"
-    origin_xyz="0 -0.13881 0.0217651" origin_rpy="0 0 0"
-    axis_xyz="0.0 1.0 0.0"
-    limit_u="${pi}" limit_l="${-pi}" limit_e="22.0" limit_v="4.4"
-  />
-  <xacro:arctos_joint
-    name="B_joint" type="revolute"
-    parent="Link_4_1" child="Link_5_1"
-    origin_xyz="0.0 -0.12543 -0.00184" origin_rpy="0 0 0"
-    axis_xyz="-1.0 0.0 0.0"
-    limit_u="1.55" limit_l="-1.55" limit_e="16.0" limit_v="3.0"
-  />
-  <xacro:arctos_joint
-    name="C_joint" type="revolute"
-    parent="Link_5_1" child="Link_6_1"
-    origin_xyz="0.0 -0.0398 0.0" origin_rpy="0 0 0"
-    axis_xyz="0.0 1.0 0.0"
-    limit_u="${pi}" limit_l="${-pi}" limit_e="16.0" limit_v="3.0"
-  />
-  <xacro:arctos_ros2_control name="arctos_interface" />
+  <xacro:arctos_arm prefix="$(arg prefix)" include_gripper="$(arg include_gripper)" />
+  <!-- Explicit legacy opt-in, not part of the Gazebo path. Jazzy hardware is
+       unvalidated. Mock/Gazebo control wrappers are supplied by later gates. -->
+  <xacro:if value="$(arg use_hardware)">
+    <xacro:include filename="$(find arctos_description)/urdf/arctos_ros2_control.xacro" />
+    <xacro:arctos_ros2_control name="arctos_interface" prefix="$(arg prefix)" />
+  </xacro:if>
 </robot>

File: arctos_description/urdf/arctos_gripper.xacro (robot description, xacro)
@@ -1,64 +1,31 @@
 <?xml version="1.0"?>
 <robot xmlns:xacro="http://www.ros.org/wiki/xacro">
-  <xacro:include filename="$(find arctos_description)/urdf/common/joint_link.xacro" />
-  <!-- Arctos Simple Pinch Gripper -->
-  <xacro:arctos_link
-    name="Gripper_1"
-    origin_xyz="0.0 0.323 -0.5685" origin_rpy="0 0 0"
-    material_name="white"
-    inertia_origin_xyz="-0.001 -0.0211 0.0" inertia_origin_rpy="0 0 0"
-    mass="0.2"
-    ixx="1e-4" iyy="1e-4" izz="1e-4" ixy="-0.0" iyz="0.0" ixz="0.0"
-  />
-  <xacro:arctos_link
-    name="Left_jaw_1"
-    origin_xyz="0.0 0.323 -0.5685" origin_rpy="0 0 0"
-    material_name="white"
-    inertia_origin_xyz="-0.0 -0.0211 0.0" inertia_origin_rpy="0 0 0"
-    mass="0."
-    ixx="0.0" iyy="0.0" izz="0.0" ixy="-0.0" iyz="0.0" ixz="0.0"
-  />
-  <xacro:arctos_link
-    name="Right_jaw_1"
-    origin_xyz="0.0 0.323 -0.5685" origin_rpy="0 0 0"
-    material_name="white"
-    inertia_origin_xyz="-0.001 -0.0211 0.0" inertia_origin_rpy="0 0 0"
-    mass="0."
-    ixx="0.0" iyy="0.0" izz="0.0" ixy="-0.0" iyz="0.0" ixz="0.0"
-  />
-  <!-- Fixed gripper joint, no axis needed -->
-  <xacro:arctos_joint
-    name="Gripper_joint" type="fixed"
-    parent="Link_6_1" child="Gripper_1"
-    origin_xyz="0.0 -0.0 0.0" origin_rpy="0 0 0"
-    limit_u="0.0" limit_l="0.0" limit_e="0.0" limit_v="0.0"
-  />
-  <!-- Left jaw joint, prismatic with axis directly defined -->
-  <!-- TODO: Movement inverted -->
-  <xacro:arctos_joint
-    name="Left_jaw_joint"
-    type="prismatic"
-    parent="Gripper_1"
-    child="Left_jaw_1"
-    origin_xyz="0.0 0.0 0.0"
-    origin_rpy="0 0 0"
-    axis_xyz="0 0 1"
-    limit_u="0.015"
-    limit_l="0.0"
-    limit_e="1.0"
-    limit_v="10.0"
-  />
-  <xacro:arctos_joint
-    name="Right_jaw_joint"
-    type="prismatic"
-    parent="Gripper_1"
-    child="Right_jaw_1"
-    origin_xyz="0.0 0.0 0.0"
-    origin_rpy="0 0 0"
-    axis_xyz="0 0 1"
-    limit_u="0.015"
-    limit_l="0.0"
-    limit_e="1.0"
-    limit_v="10.0"
-  />
+  <!-- Optional fixed attachment for visualization. Gripper actuation/contact
+       validation is a later milestone; jaws are locked at their CAD pose. -->
+  <xacro:macro name="arctos_gripper" params="prefix:=''">
+    <xacro:arctos_link name="Gripper_1" prefix="${prefix}"
+      origin_xyz="0 0.323 -0.5685" origin_rpy="0 0 0" material_name="white"
+      inertia_origin_xyz="-0.001 -0.0211 0" inertia_origin_rpy="0 0 0"
+      mass="0.2" ixx="0.0001" iyy="0.0001" izz="0.0001" ixy="0" iyz="0" ixz="0" />
+    <!-- Reference jaw properties translated into the existing mesh frame. -->
+    <xacro:arctos_link name="Left_jaw_1" prefix="${prefix}"
+      origin_xyz="0 0.323 -0.5685" origin_rpy="0 0 0" material_name="white"
+      inertia_origin_xyz="-0.003208702480352 -0.046537440309285 0.021981207372214"
+      inertia_origin_rpy="0 0 0" mass="0.073696025658594"
+      ixx="0.000011" iyy="0.000006" izz="0.000014" ixy="0.000002" iyz="0" ixz="0" />
+    <xacro:arctos_link name="Right_jaw_1" prefix="${prefix}"
+      origin_xyz="0 0.323 -0.5685" origin_rpy="0 0 0" material_name="white"
+      inertia_origin_xyz="-0.000355104952973 -0.046613535307719 -0.019237488097284"
+      inertia_origin_rpy="0 0 0" mass="0.073129021687195"
+      ixx="0.000011" iyy="0.000006" izz="0.000014" ixy="-0.000001" iyz="0" ixz="-0.000001" />
+    <joint name="${prefix}Gripper_joint" type="fixed">
+      <parent link="${prefix}tool0" /><child link="${prefix}Gripper_1" />
+    </joint>
+    <joint name="${prefix}Left_jaw_joint" type="fixed">
+      <parent link="${prefix}Gripper_1" /><child link="${prefix}Left_jaw_1" />
+    </joint>
+    <joint name="${prefix}Right_jaw_joint" type="fixed">
+      <parent link="${prefix}Gripper_1" /><child link="${prefix}Right_jaw_1" />
+    </joint>
+  </xacro:macro>
 </robot>

File: arctos_description/urdf/arctos_ros2_control.xacro (robot description, xacro)
@@ -1,72 +1,28 @@
 <?xml version="1.0"?>
 <robot xmlns:xacro="http://www.ros.org/wiki/xacro">
-  <xacro:macro name="arctos_ros2_control" params="name">
-    <xacro:include filename="$(find arctos_description)/urdf/common/joint_link.xacro"/>
-    <ros2_control name="${name}" type="system">
-      <hardware>
-        <plugin>arctos_interface/ArctosInterface</plugin>
-      </hardware>
-      <xacro:arctos_control
-        name="X_joint"
-        limit_u="${pi}" limit_l="${-pi}"
-      />
-      <xacro:arctos_control
-        name="Y_joint"
-        limit_u="-0.88" limit_l="1.97"
-      />
-      <xacro:arctos_control
-        name="Z_joint"
-        limit_u="0.65" limit_l="-1.6"
-      />
-      <joint name="A_joint">
-        <command_interface name="position">
-          <param name="min">{-2*pi}</param>
-          <param name="max">{2*pi}</param>
-        </command_interface>
-        <command_interface name="velocity">
-          <param name="min">-3.2</param>
-          <param name="max">3.2</param>
-        </command_interface>
-        <state_interface name="position">
-          <param name="initial_value">0.0</param>
-        </state_interface>
-        <state_interface name="velocity"/>
-      </joint>
-      <joint name="B_joint">
-        <command_interface name="position">
-          <param name="min">{-2*pi}</param>
-          <param name="max">{2*pi}</param>
-        </command_interface>
-        <command_interface name="velocity">
-          <param name="min">-3.2</param>
-          <param name="max">3.2</param>
-        </command_interface>
-        <state_interface name="position">
-          <param name="initial_value">0.0</param>
-        </state_interface>
-        <state_interface name="velocity"/>
-      </joint>
-      <joint name="C_joint">
-        <command_interface name="position">
-          <param name="min">{-2*pi}</param>
-          <param name="max">{2*pi}</param>
-        </command_interface>
-        <command_interface name="velocity">
-          <param name="min">-3.2</param>
-          <param name="max">3.2</param>
-        </command_interface>
-        <state_interface name="position">
-          <param name="initial_value">0.0</param>
-        </state_interface>
-        <state_interface name="velocity"/>
-      </joint>
-      <!-- <sensor name="tcp_fts_sensor">
-        <state_interface name="force.x"/>
-        <state_interface name="force.y"/>
-        <state_interface name="force.z"/>
-        <state_interface name="torque.x"/>
-        <state_interface name="torque.y"/>
-        <state_interface name="torque.z"/>
-      </sensor> -->
+  <!-- Legacy hardware adapter only. Uses the same physical bounds as geometry. -->
+  <xacro:include filename="$(find arctos_description)/urdf/common/joint_link.xacro" />
+  <xacro:macro name="arctos_hardware_joint" params="name prefix">
+    <xacro:property name="limits" value="${arctos_joint_limits[name]}" />
+    <joint name="${prefix}${name}">
+      <command_interface name="position">
+        <param name="min">${limits['lower']}</param>
+        <param name="max">${limits['upper']}</param>
+      </command_interface>
+      <state_interface name="position" />
+      <state_interface name="velocity" />
+    </joint>
+  </xacro:macro>
+  <xacro:macro name="arctos_ros2_control" params="name prefix:='' include_wrist:=true">
+    <ros2_control name="${prefix}${name}" type="system">
+      <hardware><plugin>arctos_interface/ArctosInterface</plugin></hardware>
+      <xacro:arctos_hardware_joint name="X_joint" prefix="${prefix}" />
+      <xacro:arctos_hardware_joint name="Y_joint" prefix="${prefix}" />
+      <xacro:arctos_hardware_joint name="Z_joint" prefix="${prefix}" />
+      <xacro:if value="${include_wrist}">
+        <xacro:arctos_hardware_joint name="A_joint" prefix="${prefix}" />
+        <xacro:arctos_hardware_joint name="B_joint" prefix="${prefix}" />
+        <xacro:arctos_hardware_joint name="C_joint" prefix="${prefix}" />
+      </xacro:if>
     </ros2_control>
   </xacro:macro>

File: arctos_description/urdf/base_xyz/arctos.xacro (robot description, xacro)
@@ -1,69 +1,17 @@
 <?xml version="1.0"?>
 <robot name="arctos" xmlns:xacro="http://www.ros.org/wiki/xacro">
-  <xacro:include filename="$(find arctos_description)/urdf/common/materials.xacro" />
-  <xacro:include filename="$(find arctos_description)/urdf/common/joint_link.xacro" />
-  <xacro:include filename="$(find arctos_description)/urdf/base_xyz/ros2_control.xacro" />
+  <xacro:arg name="prefix" default="" />
+  <xacro:arg name="use_hardware" default="false" />
+  <xacro:include filename="$(find arctos_description)/urdf/arctos_arm.xacro" />
   <link name="world" />
-  <joint name="world_joint" type="fixed">
-      <parent link="world"/>
-      <child link="base_link"/>
+  <joint name="$(arg prefix)world_joint" type="fixed">
+    <parent link="world" />
+    <child link="$(arg prefix)base_link" />
+    <origin xyz="0 0 0" rpy="0 0 0" />
   </joint>
-  <xacro:arctos_link
-    name="base_link"
-    origin_xyz="0 0 0" origin_rpy="0 0 0"
-    material_name="white"
-    inertia_origin_xyz="0.0009375030874740357 0.047087016508753216 0.06663230338123677"
-    inertia_origin_rpy="0 0 0"
-    mass="2.3"
-    ixx="0.0143" iyy="0.0055" izz="0.015" ixy="0.0" iyz="0.0" ixz="0.0"
-  />
-  <xacro:arctos_link
-    name="Link_1_1"
-    origin_xyz="-0.0 -0.000 -0.1126" origin_rpy="0 0 0"
-    material_name="white"
-    inertia_origin_xyz="-0.0088 -0.0005 ${0.2116-0.1126}" inertia_origin_rpy="0 0 0"
-    mass="3.0396"
-    ixx="0.0143" iyy="${0.0168*0.96536}" izz="${0.0084*0.96082}" ixy="${0.0143*-0.03956}"
-    ixz="${0.0143*-0.11546}" iyz="${0.0168*0.25198}"
-  />
-  <xacro:arctos_link
-    name="Link_2_1"
-    origin_xyz="0.0 0.020356 -0.2876" origin_rpy="0 0 0"
-    material_name="white"
-    inertia_origin_xyz="0.0042 ${-0.0098+0.020356} ${0.4174-0.2876}" inertia_origin_rpy="0 0 0"
-    mass="2.527"
-    ixx="${0.0282*0.99851}" iyy="${0.03*0.99865}" izz="${0.0063*0.99982}" ixy="${0.0282*0.05146}"
-    iyz="${0.03*-0.00591}" ixz="${0.0282*-0.01813}"
-  />
-  <xacro:arctos_link
-    name="Link_3_1"
-    origin_xyz="-0.0 0.019045 -0.54864" origin_rpy="0 0 0"
-    material_name="white"
-    inertia_origin_xyz="0.00158 -0.053 0.009" inertia_origin_rpy="0 0 0"
-    mass="0.87"
-    ixx="${0.0028*0.99944}" iyy="${0.0011*0.98426}" izz="${0.0027*0.98428}" ixy="${0.0028*-0.02203}"
-    iyz="${0.001*-0.17481}" ixz="${0.0028*0.02507}"
-  />
-  <xacro:arctos_joint
-    name="X_joint" type="revolute"
-    parent="base_link" child="Link_1_1"
-    origin_xyz="0.0 0.0 0.1126" origin_rpy="0 0 0"
-    axis_xyz="0.0 0.0 1.0"
-    limit_u="${pi}" limit_l="${-pi}" limit_e="24.3" limit_v="1.4"
-  />
-  <xacro:arctos_joint
-    name="Y_joint" type="revolute"
-    parent="Link_1_1" child="Link_2_1"
-    origin_xyz="0.0 -0.020356 ${0.2876-0.1126}" origin_rpy="0 0 0"
-    axis_xyz="-1.0 0.0 0.0"
-    limit_u="2.18" limit_l="-0.96" limit_e="270.0" limit_v="1.4"
-  />
-  <xacro:arctos_joint
-    name="Z_joint" type="revolute"
-    parent="Link_2_1" child="Link_3_1"
-    origin_xyz="0.0 0.001365 0.261035" origin_rpy="0 0 0"
-    axis_xyz="1.0 0.0 0.0"
-    limit_u="0.65" limit_l="-1.6" limit_e="97.0" limit_v="1.4"
-  />
-  <xacro:arctos_ros2_control name="arctos_interface" />
+  <xacro:arctos_arm prefix="$(arg prefix)" include_wrist="false" />
+  <xacro:if value="$(arg use_hardware)">
+    <xacro:include filename="$(find arctos_description)/urdf/arctos_ros2_control.xacro" />
+    <xacro:arctos_ros2_control name="arctos_interface" prefix="$(arg prefix)" include_wrist="false" />
+  </xacro:if>
 </robot>

File: arctos_description/urdf/base_xyz/ros2_control.xacro (robot description, xacro)
@@ -1,34 +1,8 @@
 <?xml version="1.0"?>
 <robot xmlns:xacro="http://www.ros.org/wiki/xacro">
-    <xacro:macro name="arctos_ros2_control" params="name">
-        <ros2_control name="${name}_system" type="system">
-            <hardware>
-                <plugin>arctos_interface/ArctosInterface</plugin>
-            </hardware>
-            <joint name="X_joint">
-                <command_interface name="position"/>
-                <command_interface name="velocity"/>
-                <state_interface name="position">
-                  <param name="initial_value">0</param>
-                </state_interface>
-                <state_interface name="velocity"/>
-            </joint>
-            <joint name="Y_joint">
-                <command_interface name="position"/>
-                <command_interface name="velocity"/>
-                <state_interface name="position">
-                  <param name="initial_value">0</param>
-                </state_interface>
-                <state_interface name="velocity"/>
-            </joint>
-            <joint name="Z_joint">
-                <command_interface name="position"/>
-                <command_interface name="velocity"/>
-                <state_interface name="position">
-                  <param name="initial_value">0</param>
-                </state_interface>
-                <state_interface name="velocity"/>
-            </joint>
-        </ros2_control>
-    </xacro:macro>
+  <!-- Preserve the old three-joint macro entry point without duplicating limits. -->
+  <xacro:include filename="$(find arctos_description)/urdf/arctos_ros2_control.xacro" ns="full_arm" />
+  <xacro:macro name="arctos_ros2_control" params="name prefix:=''">
+    <xacro:full_arm.arctos_ros2_control name="${name}" prefix="${prefix}" include_wrist="false" />
+  </xacro:macro>
 </robot>

File: arctos_description/urdf/common/joint_link.xacro (robot description, xacro)
@@ -1,8 +1,10 @@
 <?xml version="1.0"?>
 <robot xmlns:xacro="http://www.ros.org/wiki/xacro" name="arctos">
+  <xacro:property name="arctos_joint_limits"
+    value="${xacro.load_yaml('$(find arctos_description)/config/physical_joint_limits.yaml')}" />
   <!-- Define arctos_link macro -->
   <xacro:macro name="arctos_link"
-    params="name origin_xyz origin_rpy material_name inertia_origin_xyz inertia_origin_rpy mass ixx iyy izz ixy iyz ixz">
-    <link name="${name}">
+    params="name origin_xyz origin_rpy material_name inertia_origin_xyz inertia_origin_rpy mass ixx iyy izz ixy iyz ixz prefix:=''">
+    <link name="${prefix}${name}">
       <visual>
         <origin xyz="${origin_xyz}" rpy="${origin_rpy}" />
@@ -25,34 +27,17 @@
     </link>
   </xacro:macro>
-  <!-- Define arctos_joint macro with a default value for axis_xyz -->
-  <!-- TODO: Add param for mechanicalReduction -->
+  <!-- Geometry only: ROS control belongs in a backend wrapper. Damping is a
+       modest numerical regularization (N m s/rad), not measured gear friction. -->
   <xacro:macro name="arctos_joint"
-    params="name type parent child origin_xyz origin_rpy axis_xyz='0 0 0' limit_u limit_l limit_e limit_v">
-    <joint name="${name}" type="${type}">
-      <parent link="${parent}" />
-      <child link="${child}" />
+    params="name parent child origin_xyz origin_rpy axis_xyz prefix:='' damping:=0.1">
+    <xacro:property name="limits" value="${arctos_joint_limits[name]}" />
+    <joint name="${prefix}${name}" type="revolute">
+      <parent link="${prefix}${parent}" />
+      <child link="${prefix}${child}" />
       <origin xyz="${origin_xyz}" rpy="${origin_rpy}" />
       <axis xyz="${axis_xyz}" />
-      <limit upper="${limit_u}" lower="${limit_l}" effort="${limit_e}" velocity="${limit_v}" />
-    </joint>
-    <!-- Add transmission element -->
-    <transmission name="transmission_${name}">
-      <type>transmission_interface/SimpleTransmission</type>
-      <joint name="${name}">
-        <hardwareInterface>hardware_interface/PositionJointInterface</hardwareInterface>
-      </joint>
-      <actuator name="${name}_motor">
-        <mechanicalReduction>1.0</mechanicalReduction>
-      </actuator>
-    </transmission>
-  </xacro:macro>
-  <xacro:macro name="arctos_control" params="name limit_u limit_l">
-    <joint name="${name}">
-      <command_interface name="position">
-            <param name="min">${limit_l}</param>
-            <param name="max">${limit_u}</param>
-      </command_interface>
-      <state_interface name="position"/>
-      <state_interface name="velocity"/>
+      <limit upper="${limits['upper']}" lower="${limits['lower']}"
+        effort="${limits['effort']}" velocity="${limits['velocity']}" />
+      <dynamics damping="${damping}" friction="0.0" />
     </joint>
   </xacro:macro>
