Commit message: Basic test in gazebo

File: arctos_description/urdf/arctos_gripper.xacro (robot description, xacro)
@@ -23,4 +23,11 @@
       <parent link="${prefix}tool0" /><child link="${prefix}Gripper_1" />
     </joint>
+    <!-- Mesh-derived pad centre. +Z points out of the fingers (-Y in tool0),
+         +Y is the closing axis. Provisional until measured on the actual kit. -->
+    <link name="${prefix}grasp_frame" />
+    <joint name="${prefix}grasp_frame_joint" type="fixed">
+      <parent link="${prefix}tool0" /><child link="${prefix}grasp_frame" />
+      <origin xyz="-0.00129 -0.074 0.001367" rpy="${pi/2} 0 0" />
+    </joint>
     <joint name="${prefix}Left_jaw_joint" type="prismatic">
       <parent link="${prefix}Gripper_1" /><child link="${prefix}Left_jaw_1" />

Commit message: grab cube

File: arctos_description/urdf/arctos_gripper.xacro (robot description, xacro)
@@ -10,10 +10,10 @@
       mass="0.2" ixx="0.0001" iyy="0.0001" izz="0.0001" ixy="0" iyz="0" ixz="0" />
     <!-- Reference jaw properties translated into the existing mesh frame. -->
-    <xacro:arctos_link name="Left_jaw_1" prefix="${prefix}"
+    <xacro:arctos_link name="Left_jaw_1" prefix="${prefix}" collision_mode="jaw" pad_z="0.020367"
       origin_xyz="0 0.323 -0.5685" origin_rpy="0 0 0" material_name="white"
       inertia_origin_xyz="-0.003208702480352 -0.046537440309285 0.021981207372214"
       inertia_origin_rpy="0 0 0" mass="0.073696025658594"
       ixx="0.000011" iyy="0.000006" izz="0.000014" ixy="0.000002" iyz="0" ixz="0" />
-    <xacro:arctos_link name="Right_jaw_1" prefix="${prefix}"
+    <xacro:arctos_link name="Right_jaw_1" prefix="${prefix}" collision_mode="jaw" pad_z="-0.017633"
       origin_xyz="0 0.323 -0.5685" origin_rpy="0 0 0" material_name="white"
       inertia_origin_xyz="-0.000355104952973 -0.046613535307719 -0.019237488097284"
@@ -23,10 +23,10 @@
       <parent link="${prefix}tool0" /><child link="${prefix}Gripper_1" />
     </joint>
-    <!-- Mesh-derived pad centre. +Z points out of the fingers (-Y in tool0),
+    <!-- Simplified collision-pad centre. +Z points out of the fingers (-Y in tool0),
          +Y is the closing axis. Provisional until measured on the actual kit. -->
     <link name="${prefix}grasp_frame" />
     <joint name="${prefix}grasp_frame_joint" type="fixed">
       <parent link="${prefix}tool0" /><child link="${prefix}grasp_frame" />
-      <origin xyz="-0.00129 -0.074 0.001367" rpy="${pi/2} 0 0" />
+      <origin xyz="-0.00129 -0.066 0.001367" rpy="${pi/2} 0 0" />
     </joint>
     <joint name="${prefix}Left_jaw_joint" type="prismatic">

File: arctos_description/urdf/common/joint_link.xacro (robot description, xacro)
@@ -5,5 +5,5 @@
   <!-- Define arctos_link macro -->
   <xacro:macro name="arctos_link"
-    params="name origin_xyz origin_rpy material_name inertia_origin_xyz inertia_origin_rpy mass ixx iyy izz ixy iyz ixz prefix:=''">
+    params="name origin_xyz origin_rpy material_name inertia_origin_xyz inertia_origin_rpy mass ixx iyy izz ixy iyz ixz prefix:='' collision_mode:='mesh' pad_z:=0">
     <link name="${prefix}${name}">
       <visual>
@@ -14,4 +14,5 @@
         <material name="${material_name}" />
       </visual>
+      <xacro:if value="${collision_mode == 'mesh'}">
       <collision>
         <origin xyz="${origin_xyz}" rpy="${origin_rpy}" />
@@ -20,4 +21,17 @@
         </geometry>
       </collision>
+      </xacro:if>
+      <xacro:if value="${collision_mode == 'jaw'}">
+        <!-- Separate pad and proximal rail avoid a convex mesh hull spanning
+             the finger opening. Shared by MoveIt and Gazebo. -->
+        <collision name="pad">
+          <origin xyz="-0.00129 -0.066 ${pad_z}" rpy="0 0 0" />
+          <geometry><box size="0.018 0.016 0.008" /></geometry>
+        </collision>
+        <collision name="rail">
+          <origin xyz="-0.00129 -0.043 ${pad_z}" rpy="0 0 0" />
+          <geometry><box size="0.018 0.030 0.008" /></geometry>
+        </collision>
+      </xacro:if>
       <inertial>
         <origin xyz="${inertia_origin_xyz}" rpy="${inertia_origin_rpy}" />

File: arctos_gazebo/urdf/gazebo.urdf.xacro (robot description, xacro)
@@ -3,4 +3,8 @@
   <xacro:arg name="hardware_plugin" default="gz_ros2_control/GazeboSimSystem" />
   <xacro:include filename="$(find arctos_control)/urdf/controlled.urdf.xacro" />
+  <xacro:if value="$(arg include_gripper)">
+    <gazebo reference="Left_jaw_1"><mu1>1.0</mu1><mu2>1.0</mu2></gazebo>
+    <gazebo reference="Right_jaw_1"><mu1>1.0</mu1><mu2>1.0</mu2></gazebo>
+  </xacro:if>
   <gazebo>
     <plugin filename="gz-sim-joint-state-publisher-system" name="gz::sim::systems::JointStatePublisher">
