Commit message: update specifications using arctos studio defaults
We scraped motion limits from arctos studio web. planning and execution
now works in rviz and can be called from the moveit config package.

File: arctos_control/urdf/mock.urdf.xacro (robot description, xacro)
@@ -1,4 +1,5 @@
 <?xml version="1.0"?>
 <robot name="arctos" xmlns:xacro="http://www.ros.org/wiki/xacro">
+  <xacro:arg name="include_gripper" default="true" />
   <xacro:include filename="$(find arctos_description)/urdf/arctos.xacro" />
   <xacro:property name="initial" value="${xacro.load_yaml('$(find arctos_control)/config/initial_positions.yaml')['initial_positions']}" />
@@ -23,4 +24,18 @@
     <xacro:mock_joint name="B_joint" />
     <xacro:mock_joint name="C_joint" />
+    <xacro:if value="$(arg include_gripper)">
+      <joint name="Left_jaw_joint">
+        <command_interface name="position">
+          <param name="min">0</param><param name="max">0.015</param>
+        </command_interface>
+        <state_interface name="position"><param name="initial_value">0</param></state_interface>
+        <state_interface name="velocity" />
+      </joint>
+      <!-- GenericSystem reads the URDF mimic relation; no second actuator. -->
+      <joint name="Right_jaw_joint">
+        <state_interface name="position"><param name="initial_value">0</param></state_interface>
+        <state_interface name="velocity" />
+      </joint>
+    </xacro:if>
   </ros2_control>
 </robot>

File: arctos_description/urdf/arctos_gripper.xacro (robot description, xacro)
@@ -1,6 +1,7 @@
 <?xml version="1.0"?>
 <robot xmlns:xacro="http://www.ros.org/wiki/xacro">
-  <!-- Optional fixed attachment for visualization. Gripper actuation/contact
-       validation is a later milestone; jaws are locked at their CAD pose. -->
+  <!-- Manufacturer ROS geometry: CAD pose is open; each jaw closes 15 mm.
+       Right jaw mimics the left along the opposing axis. Units are metres.
+       Velocity/effort are simulation estimates, not servo specifications. -->
   <xacro:macro name="arctos_gripper" params="prefix:=''">
     <xacro:arctos_link name="Gripper_1" prefix="${prefix}"
@@ -22,9 +23,16 @@
       <parent link="${prefix}tool0" /><child link="${prefix}Gripper_1" />
     </joint>
-    <joint name="${prefix}Left_jaw_joint" type="fixed">
+    <joint name="${prefix}Left_jaw_joint" type="prismatic">
       <parent link="${prefix}Gripper_1" /><child link="${prefix}Left_jaw_1" />
+      <axis xyz="0 0 -1" />
+      <limit lower="0" upper="0.015" velocity="0.02" effort="20" />
+      <dynamics damping="0.1" friction="0" />
     </joint>
-    <joint name="${prefix}Right_jaw_joint" type="fixed">
+    <joint name="${prefix}Right_jaw_joint" type="prismatic">
       <parent link="${prefix}Gripper_1" /><child link="${prefix}Right_jaw_1" />
+      <axis xyz="0 0 1" />
+      <limit lower="0" upper="0.015" velocity="0.02" effort="20" />
+      <mimic joint="${prefix}Left_jaw_joint" multiplier="1" offset="0" />
+      <dynamics damping="0.1" friction="0" />
     </joint>
   </xacro:macro>

Commit message: first gazebo integration

File: arctos_control/urdf/mock.urdf.xacro (robot description, xacro)
@@ -1,41 +1,4 @@
 <?xml version="1.0"?>
 <robot name="arctos" xmlns:xacro="http://www.ros.org/wiki/xacro">
-  <xacro:arg name="include_gripper" default="true" />
-  <xacro:include filename="$(find arctos_description)/urdf/arctos.xacro" />
-  <xacro:property name="initial" value="${xacro.load_yaml('$(find arctos_control)/config/initial_positions.yaml')['initial_positions']}" />
-  <xacro:macro name="mock_joint" params="name">
-    <joint name="${name}">
-      <command_interface name="position">
-        <param name="min">${arctos_joint_limits[name]['lower']}</param>
-        <param name="max">${arctos_joint_limits[name]['upper']}</param>
-      </command_interface>
-      <state_interface name="position">
-        <param name="initial_value">${initial[name]}</param>
-      </state_interface>
-      <state_interface name="velocity" />
-    </joint>
-  </xacro:macro>
-  <ros2_control name="ArctosMock" type="system">
-    <hardware><plugin>mock_components/GenericSystem</plugin></hardware>
-    <xacro:mock_joint name="X_joint" />
-    <xacro:mock_joint name="Y_joint" />
-    <xacro:mock_joint name="Z_joint" />
-    <xacro:mock_joint name="A_joint" />
-    <xacro:mock_joint name="B_joint" />
-    <xacro:mock_joint name="C_joint" />
-    <xacro:if value="$(arg include_gripper)">
-      <joint name="Left_jaw_joint">
-        <command_interface name="position">
-          <param name="min">0</param><param name="max">0.015</param>
-        </command_interface>
-        <state_interface name="position"><param name="initial_value">0</param></state_interface>
-        <state_interface name="velocity" />
-      </joint>
-      <!-- GenericSystem reads the URDF mimic relation; no second actuator. -->
-      <joint name="Right_jaw_joint">
-        <state_interface name="position"><param name="initial_value">0</param></state_interface>
-        <state_interface name="velocity" />
-      </joint>
-    </xacro:if>
-  </ros2_control>
+  <xacro:include filename="$(find arctos_control)/urdf/controlled.urdf.xacro" />
 </robot>
